File: 02_Elements/LWK2_MainBoard_Rev_1/03_Mechanics/LWK2_MainBoard_Rev_1_Housing.brd (EAGLE design)
At the start: 60 x 139 mm, 32 parts

Commit message: Further Development
Updated:
- Final HW of LWK2_MainBoard_Rev_1
- Final Housing of LWK2_MainBoard_Rev_1 (print with MDF 2MM)
- Cleaned folders
- Added photos for the WIKI
Parts:
- removed C_LCD: 1u, resistor:C1206
- removed C_VR_0, C_VR_1: 10uF, resistor:C1206
- removed J_AEXT_0, J_AEXT_1, J_LED, J_SWEXT: KLBR4, con-lumberg:KLBR4
- removed J_BHT: 22-05-7048-04, con-molex:7395-04
- removed Q_BZZ: (no value), microbuilder:SOT23-WIDE
- removed R_BZZ: (no value), resistor:R1206
- removed R_DATA: 470Ohm, resistor:R1206
- removed R_LCD_0, R_LCD_1, R_VR_0: 0, resistor:R1206
- removed R_SW_0, R_SW_1, R_SW_2, R_SW_EXT: 10k, resistor:R1206
- removed R_VR_1: 121, resistor:R1206
- removed SWPAD_0, SWPAD_1, SWPAD_2, SWPAD_3: (no value), PdMM_Aux:MDM_V3_LEDPAD
- removed SW_0, SW_1, SW_2: (no value), adafruit:B3F-40XX-ROUND
- removed U_ADXL345: (no value), PdMM_Aux:GY-291_ADXL345
- removed U_ARDUINO: ARDUINO-MEGA_LWK2_CLEAN, SparkFun-Boards:ARDUINO_MEGA_LWK2_CLEAN
- removed U_BZZ: BUZZERSMD, SparkFun:BUZZER-CMT1603
- removed U_LCD: NOKIA5110, _LCD_Nokia5110:NOKIA5110
- removed U_SDSOCKET: CATALEX_MICROSDSOCKET_SMD, PdMM_Aux:CATALEX_MICROSDSOCKET_SMD
- removed U_VR: LM1086TO263, v-reg-2:TO263
Connections:
- removed net 3V3: U_ARDUINO.P3V3
- removed net 3V3_ARD: R_LCD_1.1
- removed net 5V_ARD: J_AEXT_0.S, J_AEXT_1.S, J_BHT.1, R_LCD_0.1, R_SW_0.1, R_SW_1.1, R_SW_2.1, R_SW_EXT.1, U_ADXL345.2, U_ARDUINO.P5V0, U_BZZ.P$1, U_SDSOCKET.2
- removed net 5V_LED: C_VR_1.1, J_LED.S, R_VR_1.1, SWPAD_0.2, SWPAD_1.2, SWPAD_2.2, SWPAD_3.2
- removed net ACC_SCL: U_ADXL345.8, U_ARDUINO.P21
- removed net ACC_SDA: U_ADXL345.7, U_ARDUINO.P20
- removed net AEXT_0: J_AEXT_0.T, U_ARDUINO.PA6
- removed net AEXT_1: J_AEXT_1.T, U_ARDUINO.PA7
- removed net BHT_RX: J_BHT.3, U_ARDUINO.P0
- removed net BHT_TX: J_BHT.4, U_ARDUINO.P1
- removed net BUZZ: R_BZZ.2, U_ARDUINO.P16
- removed net CS: U_ADXL345.3
- removed net GND: C_LCD.2, C_VR_0.2, C_VR_1.2, J_AEXT_0.B, J_AEXT_0.R, J_AEXT_1.B, J_AEXT_1.R, J_BHT.2, J_LED.B, J_LED.R, J_SWEXT.B, J_SWEXT.R, Q_BZZ.3, R_VR_0.1, SWPAD_0.3, SWPAD_1.3, SWPAD_2.3, SWPAD_3.3, SW_0.3, SW_1.3, SW_2.3, U_ADXL345.1, U_ARDUINO.PGND1, U_ARDUINO.PGND2, U_ARDUINO.PGND3, U_ARDUINO.PGND4, U_LCD.8, U_SDSOCKET.1
- removed net INT1: U_ADXL345.4
- removed net INT2: U_ADXL345.5
- removed net LCD_BCKL: U_ARDUINO.P15, U_LCD.7
- removed net LCD_CE: U_ARDUINO.P4, U_LCD.2
- removed net LCD_CLK: U_ARDUINO.P7, U_LCD.5
- removed net LCD_DC: U_ARDUINO.P5, U_LCD.3
- removed net LCD_DIN: U_ARDUINO.P6, U_LCD.4
- removed net LCD_PW: C_LCD.1, R_LCD_0.2, R_LCD_1.2, U_LCD.6
- removed net LCD_RST: U_ARDUINO.P3, U_LCD.1
- removed net LED: R_DATA.1, U_ARDUINO.P2
- removed net LED_0: R_DATA.2, SWPAD_0.5
- removed net LED_1: SWPAD_0.1, SWPAD_1.5
- removed net LED_2: SWPAD_1.1, SWPAD_2.5
- removed net LED_3: SWPAD_2.1, SWPAD_3.5
- removed net LED_STR: J_LED.T, SWPAD_3.1
- removed net N$1: R_VR_0.2, U_VR.1
- removed net N$2: R_VR_1.2, U_VR.2
- removed net N$4: Q_BZZ.2, U_BZZ.P$2
- removed net N$8: Q_BZZ.1, R_BZZ.1
- removed net SDO: U_ADXL345.6
- removed net SD_CS: U_ARDUINO.P44, U_SDSOCKET.6
- removed net SD_MISO: U_ARDUINO.P50, U_SDSOCKET.3
- removed net SD_MOSI: U_ARDUINO.P51, U_SDSOCKET.4
- removed net SD_SCK: U_ARDUINO.P52, U_SDSOCKET.5
- removed net SWPAD_0: SWPAD_0.4, U_ARDUINO.PA2
- removed net SWPAD_1: SWPAD_1.4, U_ARDUINO.PA3
- removed net SWPAD_2: SWPAD_2.4, U_ARDUINO.PA4
- removed net SWPAD_3: SWPAD_3.4, U_ARDUINO.PA5
- removed net SW_0: R_SW_0.2, SW_0.1, U_ARDUINO.P19
- removed net SW_1: R_SW_1.2, SW_1.1, U_ARDUINO.P18
- removed net SW_2: R_SW_2.2, SW_2.1, U_ARDUINO.P17
- removed net SW_EXT: J_SWEXT.S, J_SWEXT.T, R_SW_EXT.2, U_ARDUINO.P14
- removed net VIN: C_VR_0.1, U_ARDUINO.PVIN, U_VR.3
Routing:
- removed copper zone on layer 1, net GND
- removed copper zone on layer 16, net GND
- removed copper zone on layer 16, net N$3
Other:
- board size 60 x 139 mm -> 6 x 6 mm
- board text added: "ANALOG SENSOR 0"
- board text added: "ANALOG SENSOR 1"
- board text added: "Check BanaNut Electronics Github!"
- board text added: "Developed by Pablo dMM Pablodmm.isp@gmail.com Madrid, Spain 2018"
- board text added: "LED CON"
- board text added: "LIGHTWAND KOSMONAUT V.2"
- board text added: "LightWand Kosmonaut V2 is an Open Source project with a CC BY-NC-SA License."
- board text added: "PW 7.4V"
- board text added: "SD CARD SOCKET"
- board text added: "SD SOCKET"
- board text added: "SWPAD_0"
- board text added: "SWPAD_1"
- board text added: "SWPAD_2"
- board text added: "SWPAD_3"
- board text added: "SW_CON"
- board text added: "TO ANALOG SENSOR 0"
- board text added: "TO ANALOG SENSOR 1"
- board text added: "TO LED STRIPE"
- board text added: "USB CON"
- board text removed: "C_LCD"
- board text removed: "C_VR_0"
- board text removed: "C_VR_1"
- board text removed: "J_AEXT_0"
- board text removed: "J_AEXT_1"
- board text removed: "J_BTH"
- board text removed: "J_LED"
- board text removed: "J_SWEXT"
- board text removed: "LIGHTWAND KOSMONAUT V2"
- board text removed: "LIGHTWAND KOSMONAUT V2 is the second versión of the LIGHTWAND KOSMONAUT. Designed by Pablo dMM(Pablodmm.isp@gmail.com), based on the Michael Ross original LightWand"
- board text removed: "LWK2_MainBoard_Rev_1"
- board text removed: "Q_BUZZ"
- board text removed: "R_BUZZ"
- board text removed: "R_DATA"
- board text removed: "R_LCD_0"
- board text removed: "R_LCD_1"
- board text removed: "R_SWEXT"
- board text removed: "R_SW_0"
- board text removed: "R_SW_1"
- board text removed: "R_SW_2"
- board text removed: "R_VR_0"
- board text removed: "R_VR_1"
- board text removed: "SD CARD SOCKET BELOW"
- board text removed: "Spain 2018"
- board text removed: "U_BUZZ"
- board text removed: "U_VR"
- board text removed: "VCC GND TX RX"

Commit message: Documentation Update
New product photos and refurbished yet still not finished 3D model
Other:
- board size 6 x 6 mm -> 250.5 x 143 mm
